Commit message: JEPA datagen

File: assets/mini_pupper/mini_pupper.urdf (robot description, URDF)
Before this commit: robot mini_pupper, 17 links, 16 joints
Links:
- added link camera_link, mass 0.01; visual box size=0.01 0.02 0.02
Joints:
- added joint camera_joint: type fixed, parent base_link, child camera_link, origin xyz=0.09055 0 0.07000 rpy=0 0.26180 0
